File: RocketBoard.kicad_pcb (KiCad board)
At the start: 2 copper layers, 8 parts, among them SW1 GT-TC063F-H035-L30, U1 ATSAMD21G18A-AU, U2 LSM6DS3TR, U3 MS561101BA03-50, U4 W25Q64JVSSIQ, U5 AP2112K-3.3

Commit message: routing start
Parts:
- removed U3: MS561101BA03-50, footprints:SON8_MS5611_TEC
- added C1: 100nF, Capacitor_SMD:C_0603_1608Metric, F.Cu at (170.0, 114.9)
- added C10: 100nF, Capacitor_SMD:C_0603_1608Metric, F.Cu at (174.0, 117.4)
- added C11: 0.47uF, Capacitor_SMD:C_0603_1608Metric, F.Cu at (174.0, 119.9)
- added C12: 10nF, Capacitor_SMD:C_0402_1005Metric, F.Cu at (181.5, 116.6)
- added C13: 100nF, Capacitor_SMD:C_0603_1608Metric, F.Cu at (174.0, 122.4)
- added C14: 100nF, Capacitor_SMD:C_0603_1608Metric, F.Cu at (174.0, 124.9)
- added C15: 1uF, Capacitor_SMD:C_0402_1005Metric, F.Cu at (181.5, 118.6)
- added C16: 1uF, Capacitor_SMD:C_0402_1005Metric, F.Cu at (181.5, 120.5)
- added C17: 20pF, Capacitor_SMD:C_0603_1608Metric, F.Cu at (174.0, 127.5)
- added C18: 20pF, Capacitor_SMD:C_0603_1608Metric, F.Cu at (178.1, 114.9)
- added C19: 100nF, Capacitor_SMD:C_0603_1608Metric, F.Cu at (178.1, 117.4)
- added C2: 1uF, Capacitor_SMD:C_0402_1005Metric, F.Cu at (181.5, 114.6)
- added C20: 100nF, Capacitor_SMD:C_0603_1608Metric, F.Cu at (178.1, 119.9)
- added C21: 100nF, Capacitor_SMD:C_0603_1608Metric, F.Cu at (178.1, 122.4)
- added C22: 100nF, Capacitor_SMD:C_0603_1608Metric, F.Cu at (178.1, 124.9)
- added C3: 100nF, Capacitor_SMD:C_0603_1608Metric, F.Cu at (170.0, 117.4)
- added C4: 10uF, Capacitor_SMD:C_0603_1608Metric, F.Cu at (170.0, 119.9)
- added C5: 100nF, Capacitor_SMD:C_0603_1608Metric, F.Cu at (170.0, 122.4)
- added C6: 100nF, Capacitor_SMD:C_0603_1608Metric, F.Cu at (170.0, 124.9)
- added C7: 100nF, Capacitor_SMD:C_0603_1608Metric, F.Cu at (170.0, 127.5)
- added C9: 2.2uF, Capacitor_SMD:C_0603_1608Metric, F.Cu at (174.0, 114.9)
- added D2: BLUE, LED_SMD:LED_0402_1005Metric, F.Cu at (181.1, 129.7)
- added D3: RED, LED_SMD:LED_0402_1005Metric, F.Cu at (181.1, 131.7)
- added H1: MountingHole, MountingHole:MountingHole_3mm, F.Cu at (141.9, 126.9)
- added H2: MountingHole, MountingHole:MountingHole_3mm, F.Cu at (142.0, 102.9)
- added H3: MountingHole, MountingHole:MountingHole_3mm, F.Cu at (103.1, 126.9)
- added H4: MountingHole, MountingHole:MountingHole_3mm, F.Cu at (103.1, 103.1)
- added J2: USB_B_Micro, Connector_USB:USB_Micro-B_Amphenol_10103594-0001LF_Horizontal, F.Cu at (112.5, 102.5)
- added J3: Conn_01x03_Pin, Connector_PinHeader_2.54mm:PinHeader_1x03_P2.54mm_Vertical, F.Cu at (131.7, 103.6)
- added J4: Conn_01x03_Pin, Connector_PinHeader_2.54mm:PinHeader_1x03_P2.54mm_Vertical, F.Cu at (135.8, 103.6)
- added J5: Conn_02x03_Counter_Clockwise, Connector_PinHeader_2.54mm:PinHeader_2x03_P2.54mm_Vertical, F.Cu at (107.8, 118.1)
- added R10: 100K, Resistor_SMD:R_0603_1608Metric, F.Cu at (195.0, 119.0)
- added R2: 100K, Resistor_SMD:R_0603_1608Metric, F.Cu at (195.0, 101.5)
- added R3: 100K, Resistor_SMD:R_0603_1608Metric, F.Cu at (195.0, 104.0)
- added R4: 100K, Resistor_SMD:R_0603_1608Metric, F.Cu at (195.0, 106.5)
- added R6: 100K, Resistor_SMD:R_0603_1608Metric, F.Cu at (195.0, 109.0)
- added R7: 330R, Resistor_SMD:R_0603_1608Metric, F.Cu at (195.0, 111.5)
- added R8: 330R, Resistor_SMD:R_0603_1608Metric, F.Cu at (195.0, 114.0)
- added R9: 10K, Resistor_SMD:R_0603_1608Metric, F.Cu at (195.0, 116.5)
- moved SW1 74.7 mm to (104.8, 112.0)
- moved D1 48.4 mm to (116.5, 110.6), turned to 180 degrees
- moved U4 43.4 mm to (121.9, 104.4), turned to -90 degrees
- moved U1 41.8 mm to (119.1, 120.9)
- moved R1 30.1 mm to (131.4, 121.2)
- moved U2 22.0 mm to (137.9, 121.4)
- moved U5 21.2 mm to (151.5, 126.0)
Connections:
- net Net-(R8-Pad1) renamed /SWD_RESET
- U1 pad 4: unconnected-(U1-PA03-Pad4) -> /USR_LED
- U1 pad 45: unconnected-(U1-PA30-Pad45) -> /SWCLK
- U1 pad 46: unconnected-(U1-PA31-Pad46) -> /SWDIO
- U1 pad 7: /USR_LED -> /PWM1
- U1 pad 8: unconnected-(U1-PB09-Pad8) -> /PWM2
Other:
- board outline added: 45 x 30 mm

Commit message: started placing things
Parts:
- added C23: 1uF, Capacitor_SMD:C_0402_1005Metric, F.Cu at (110.6, 136.4)
- added C8: 1uF, Capacitor_SMD:C_0402_1005Metric, F.Cu at (110.6, 142.6)
- added Card1: TF-102-15, easyeda2kicad:TF-SMD_TF-102-15, F.Cu at (130.3, 140.7)
- added LED1: WS2812B-MINI, easyeda2kicad:LED-SMD_4P-L3.5-W3.5-TL_WS2812B, B.Cu at (121.8, 117.3)
- added TP1: TestPoint, TestPoint:TestPoint_Pad_3.0x3.0mm, B.Cu at (120.9, 104.8)
- added TP2: TestPoint, TestPoint:TestPoint_Pad_3.0x3.0mm, B.Cu at (126.4, 104.8)
- added U3: MMZ2012R601AT000, easyeda2kicad:L0805, F.Cu at (113.9, 134.4)
- added U6: BMP388, easyeda2kicad:SENSORM-SMD_BMP388, F.Cu at (117.9, 141.5)
- added U7: L78L05ABUTR, easyeda2kicad:SOT-89-3_L4.5-W2.5-P1.50-LS4.2-TL, F.Cu at (110.0, 139.6)
- added X1: X201232768KLD2SI, easyeda2kicad:OSC-SMD_L2.0-W1.2, F.Cu at (114.4, 130.6)
- moved R9 71.5 mm to (123.8, 109.7), turned to 180 degrees
- moved R7 70.4 mm to (127.3, 130.8)
- moved C18 68.2 mm to (111.9, 131.3), turned to 180 degrees
- moved C20 66.2 mm to (112.0, 116.0), turned to 90 degrees
- moved C22 64.2 mm to (115.6, 139.8), turned to -90 degrees
- moved D3 63.9 mm to (121.2, 109.7)
- moved C16 63.3 mm to (118.6, 113.3), turned to 90 degrees
- moved C17 62.1 mm to (112.0, 129.7), turned to 180 degrees
- moved C21 60.6 mm to (120.7, 141.7), turned to -90 degrees
- moved C5 57.2 mm to (112.9, 126.1), turned to 180 degrees
- moved C4 54.5 mm to (118.4, 137.2)
- moved C7 54.0 mm to (122.9, 101.1), turned to 180 degrees
- moved D2 53.9 mm to (127.3, 132.2)
- moved C6 53.4 mm to (117.0, 119.1), turned to 180 degrees
- moved C3 52.3 mm to (119.9, 132.2), turned to 180 degrees
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Connections:
- U1 pad 47: unconnected-(U1-PB02-Pad47) -> /RGB_LED_IN
- U4 pad 8: Net-(U4-IO3) -> +3.3V
Other:
- board size 45 x 30 mm -> 45 x 50 mm
- copper layers 2 -> 4

Commit message: routed?
Parts:
- moved R8 83.8 mm to (111.3, 119.1)
- moved R10 81.3 mm to (117.7, 144.5), turned to -90 degrees
- moved C2 69.4 mm to (112.8, 124.2), turned to 180 degrees
- moved R6 69.3 mm to (129.9, 133.0), turned to 180 degrees
- moved R2 68.9 mm to (126.7, 111.0)
- moved R3 67.2 mm to (127.8, 102.2), turned to 180 degrees
- moved C15 61.6 mm to (120.7, 109.0), turned to 180 degrees
- moved R4 58.3 mm to (136.7, 106.0), turned to 90 degrees
- moved C12 53.0 mm to (128.5, 119.4), turned to 90 degrees
- moved J4 46.3 mm to (103.9, 137.2), turned to 180 degrees
- moved C8 44.8 mm to (140.3, 109.1), turned to 0 degrees
- moved U7 41.3 mm to (140.9, 112.2), turned to 0 degrees
- moved J3 41.1 mm to (108.0, 137.2), turned to 180 degrees
- moved C23 36.4 mm to (140.3, 115.4), turned to 0 degrees
- moved C7 11.4 mm to (134.2, 102.2), turned to 0 degrees
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Connections:
- C20 pad 1: +3.3V -> /RESET
- J5 pad 6: unconnected-(J5-Pin_6-Pad6) -> GND
- R8 pad 2: +3.3V -> /RESET
- U1 pad 40: +3.3V -> /RESET
Routing:
- net GND: track 0.00 -> 129.3 mm, vias 0 -> 25
- net +3.3V: track 0.00 -> 68.5 mm, vias 0 -> 16
- net VBUS: track 0.00 -> 43.4 mm, vias 0 -> 3
- net /GYRO_SCK: track 0.00 -> 32.9 mm
- net /GYRO1_CS: track 0.00 -> 29.2 mm, vias 0 -> 2
- net /ALT_MISO: track 0.00 -> 29.0 mm
- net /PWM2: track 0.00 -> 26.4 mm
- net /FLASH_CS: track 0.00 -> 25.1 mm
- net /GYRO1_INT: track 0.00 -> 22.5 mm, vias 0 -> 2
- net /GYRO_MOSI: track 0.00 -> 22.5 mm, vias 0 -> 2
- net +5V: track 0.00 -> 21.2 mm, vias 0 -> 1
- net /SD_MISO: track 0.00 -> 20.4 mm
- net /USB_D-: track 0.00 -> 20.1 mm
- net /USB_D+: track 0.00 -> 20.1 mm
- net /ALT_CS: track 0.00 -> 20.1 mm
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- added copper zone on In2.Cu, net +3.3V
- added copper zone on In1.Cu, net GND
Other:
- outline, holes or cut-outs redrawn
- board text added: "+"
- board text added: "-"
- board text added: "X+"
- board text added: "Y+"
- board text added: "Z+"
