File: RocketBoard.kicad_sch (KiCad schematic)
At the start: 47 parts, among them J1 Micro_SD_Card, J2 USB_B_Micro, J3 Conn_01x03_Pin, J4 Conn_01x03_Pin, SW1 GT-TC063F-H035-L30, U1 ATSAMD21G18A-AU, U2 LSM6DS3TR, U4 W25Q64JVSSIQ, U5 AP2112K-3.3, U6 BMP388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

Commit message: routing start
Parts:
- removed TP1, TP2: TestPoint, symbol Connector:TestPoint
- added H1, H2, H3, H4: MountingHole, symbol Mechanical:MountingHole
- added J5: Conn_02x03_Counter_Clockwise, Connector_PinHeader_2.54mm:PinHeader_2x03_P2.54mm_Vertical, symbol Connector_Generic:Conn_02x03_Counter_Clockwise
- C1, C10, C11, C13, C14, C17, C18, C19, C20, C21, C22, C3, C4, C5, C6, C7, C9: footprint (none) -> Capacitor_SMD:C_0603_1608Metric
- C12, C15, C16, C2: footprint (none) -> Capacitor_SMD:C_0402_1005Metric
- D2, D3: footprint (none) -> LED_SMD:LED_0402_1005Metric
- J2: footprint (none) -> Connector_USB:USB_Micro-B_Amphenol_10103594-0001LF_Horizontal
- J3, J4: footprint (none) -> Connector_PinHeader_2.54mm:PinHeader_1x03_P2.54mm_Vertical
- R10, R2, R3, R4, R6, R7, R8, R9: footprint (none) -> Resistor_SMD:R_0603_1608Metric
Connections:
- net +3.3V: now also J5.5 (Pin_5)
- net GND: now also J5.4 (Pin_4)
- net SWCLK: now also J5.1 (Pin_1)
- net SWDIO: now also J5.2 (Pin_2)
- net SWD_RESET: now reaches R8.1, SW1.3, SW1.4
- net SWD_RESET: now also J5.3 (Pin_3)
- no-connect marks 34 -> 35
Other:
- note added: "PWM Output"
- note added: "SWD Header"
- moved on the sheet: C20, J3, J4, R8, SW1

Commit message: started placing things
Parts:
- removed FB1: FerriteBead, symbol Device:FerriteBead
- removed J1: Micro_SD_Card, symbol Connector:Micro_SD_Card
- removed Y1: 32.768 kHz, symbol Device:Crystal
- added C23, C8: 1uF, Capacitor_SMD:C_0402_1005Metric, symbol Device:C
- added Card1: TF-102-15, easyeda2kicad:TF-SMD_TF-102-15, symbol easyeda2kicad:TF-102-15
- added LED1: WS2812B-MINI, easyeda2kicad:LED-SMD_4P-L3.5-W3.5-TL_WS2812B, symbol easyeda2kicad:WS2812B-MINI
- added TP1, TP2: TestPoint, TestPoint:TestPoint_Pad_3.0x3.0mm, symbol Connector:TestPoint
- added U3: MMZ2012R601AT000, easyeda2kicad:L0805, symbol easyeda2kicad:MMZ2012R601AT000
- added U7: L78L05ABUTR, easyeda2kicad:SOT-89-3_L4.5-W2.5-P1.50-LS4.2-TL, symbol easyeda2kicad:L78L05ABUTR
- added X1: X201232768KLD2SI, easyeda2kicad:OSC-SMD_L2.0-W1.2, symbol easyeda2kicad:X201232768KLD2SI
- H1, H2, H3, H4: footprint (none) -> MountingHole:MountingHole_3mm
Connections:
- net +3.3V: now also U4.8 (VCC), Card1.4 (VDD), U3.2
- net GND: now also C23.2, C8.2, Card1.10 (SHELL), Card1.11 (SHELL), Card1.12 (SHELL), Card1.6 (VSS), Card1.9 (SHELL), LED1.3 (VSS), TP2.1, U7.2 (GND)
- net SD_CS: now also Card1.2 (CD/DAT3)
- net SD_MISO: now also Card1.7 (DAT0)
- net SD_MOSI: now also Card1.3 (CMD)
- net SD_SCK: now also Card1.5 (CLK)
- net VBUS: now also C23.1, TP1.1, U7.3 (VIN)
- net XIN_32: now also X1.1 (OSC1)
- net XOUT_32: now also X1.2 (OSC2)
- net at C3.1, C4.1, U1.6 (VDDANA): now also U3.1
- net RGB_LED_IN: now reaches U1.47 (PB02)
- net RGB_LED_IN: now also LED1.4 (DIN)
- net at R4.2, U4.7 (IO3): no longer U4.8 (VCC)
- new net +5V: C8.1, LED1.1 (VDD), U7.1 (VOUT)
Other:
- note added: "Batt. Pads"
- note added: "Check if can be normal io pin or not"
- note added: "Mounting"
- note added: "SWD"
- note added: "USB"
- moved on the sheet: C1, C17, C18, C19, C2, C20, C3, C4, C5, C6, D1, D2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

Commit message: routed?
Connections:
- net +3.3V: no longer C20.1, R8.2, U1.40 (~{RESET})
- net GND: now also J5.6 (Pin_6)
- new net RESET: C20.1, R8.2, U1.40 (~{RESET})
- no-connect marks 35 -> 34
Changed lines of the file:
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@@
   (junction (at 60.96 92.075) (diameter 0) (color 0 0 0 0)
   )
-  (junction (at 60.325 39.37) (diameter 0) (color 0 0 0 0)
-  )
   (junction (at 196.85 238.76) (diameter 0) (color 0 0 0 0)
   )
@@
   )
   (junction (at 126.365 228.6) (diameter 0) (color 0 0 0 0)
+  )
+  (junction (at 200.025 170.815) (diameter 0) (color 0 0 0 0)
   )
   (junction (at 256.54 107.315) (diameter 0) (color 0 0 0 0)
@@
   (no_connect (at 111.76 59.055))
   (no_connect (at 114.3 59.055))
-  (no_connect (at 198.12 165.735))
   (no_connect (at 182.245 223.52))
   (no_connect (at 320.04 141.605))
@@
     (stroke (width 0) (type default))
   )
+  (wire (pts (xy 200.025 165.735) (xy 200.025 170.815))
+    (stroke (width 0) (type default))
+  )
   (wire (pts (xy 245.11 213.995) (xy 245.11 216.535))
     (stroke (width 0) (type default))
@@
     (stroke (width 0) (type default))
   )
+  (wire (pts (xy 198.12 165.735) (xy 200.025 165.735))
+    (stroke (width 0) (type default))
+  )
   (wire (pts (xy 178.435 170.815) (xy 185.42 170.815))
     (stroke (width 0) (type default))
@@
     (stroke (width 0) (type default))
   )
-  (wire (pts (xy 60.325 29.845) (xy 60.325 39.37))
-    (stroke (width 0) (type default))
-  )
   (wire (pts (xy 127 117.475) (xy 127 125.73))
     (stroke (width 0) (type default))
@@
     (stroke (width 0) (type default))
   )
+  (wire (pts (xy 200.025 170.815) (xy 201.93 170.815))
+    (stroke (width 0) (type default))
+  )
   (wire (pts (xy 42.545 47.625) (xy 42.545 44.45))
     (stroke (width 0) (type default))
@@
     (stroke (width 0) (type default))
   )
-  (wire (pts (xy 60.325 39.37) (xy 66.04 39.37))
+  (wire (pts (xy 58.42 39.37) (xy 66.04 39.37))
     (stroke (width 0) (type default))
   )
@@
     (stroke (width 0) (type default))
   )
-  (wire (pts (xy 198.12 170.815) (xy 201.93 170.815))
+  (wire (pts (xy 198.12 170.815) (xy 200.025 170.815))
     (stroke (width 0) (type default))
   )
@@
   )
   (wire (pts (xy 319.405 83.82) (xy 319.405 75.565))
-    (stroke (width 0) (type default))
-  )
-  (wire (pts (xy 58.42 39.37) (xy 60.325 39.37))
     (stroke (width 0) (type default))
   )
@@
         )
       )
-    )
-  )
-  (symbol (lib_id "power:+3.3V") (at 60.325 29.845 0) (unit 1)
-    (in_bom yes) (on_board yes) (dnp no) (fields_autoplaced)
-    (property "Reference" "#PWR034" (at 60.325 33.655 0)
-      (effects (font (size 1.27 1.27)) hide)
-    )
-    (property "Value" "+3.3V" (at 60.325 25.4 0)
-      (effects (font (size 1.27 1.27)))
-    )
-    (property "Footprint" "" (at 60.325 29.845 0)
-      (effects (font (size 1.27 1.27)) hide)
-    )
-    (property "Datasheet" "" (at 60.325 29.845 0)
-      (effects (font (size 1.27 1.27)) hide)
-    )
-    (pin "1")
-    (instances
-      (project "RocketBoard"
-        (path "/7bdfbe8f-135e-4c79-9173-5900f6783fbe"
-          (reference "#PWR034") (unit 1)
-        )
-      )
